Commit message: latest

File: turtlebot3_description/urdf/turtlebot3_waffle_naked.urdf.xacro (robot description, xacro)
@@ -200,5 +200,5 @@
     </inertial>-->
   </link>
-  <joint name="camera_rgb_joint" type="fixed">
+  <!--joint name="camera_rgb_joint" type="fixed">
     <origin xyz="${r200_cam_rgb_px} ${r200_cam_rgb_py} ${r200_cam_rgb_pz}" rpy="0 0 0"/>
     <parent link="camera_link"/>
@@ -223,4 +223,30 @@
     <child link="camera_depth_optical_frame"/>
   </joint>
-  <link name="camera_depth_optical_frame"/>
+  <link name="camera_depth_optical_frame"/-->
+  <material name="Kinect2Grey">
+	  <color rgba="0.15 0.15 0.15 1.0"/>
+  </material>
+  <!-- Joint connecting the parent to our frame_in -->
+  <joint name="${prefix}_kinect2_in_joint" type="fixed">
+	  <origin xyz="0 0 0" rpy="0 0 0"/>
+	  <parent link="$camera_link"/>
+	  <child link="${prefix}_kinect2_rgb_optical_frame"/>
+  </joint>
+  <link name="${prefix}_kinect2_rgb_optical_frame">
+	  <visual>
+		  <origin rpy="0 0 0" xyz="0 0 0"/>
+		  <geometry>
+			  <!-- these meshes were exported in mm, so scale back to m -->
+			  <mesh filename="package://iai_kinect2_description/meshes/kinect2_origin_on_rgb_optical_frame.stl" scale="0.001 0.001 0.001"/>
+		  </geometry>
+		  <material name="Kinect2Grey"/>
+	  </visual>
+	  <collision>
+		  <origin xyz="0 0 0" rpy="0 0 0" />
+		  <geometry>
+			  <mesh
+				  filename="package://iai_kinect2_description/meshes/kinect2_origin_on_rgb_optical_frame.stl" scale="0.001 0.001 0.001"/>
+		  </geometry>
+	  </collision>
+  </link>
 </robot>
